File: Connectors.kicad_sch (KiCad schematic)
At the start: 5 parts, among them J1 282836-5, J2 1725669, J3 53398-0567

Commit message: połączenie ścieżkami, wylanie masy
Parts:
- C16, C17: footprint Capacitor_SMD:C_0201_0603Metric -> Capacitor_SMD:C_0603_1608Metric_Pad1.08x0.95mm_HandSolder
Changed lines of the file:
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@@
 			)
 		)
-		(property "Footprint" "Capacitor_SMD:C_0201_0603Metric"
+		(property "Footprint" "Capacitor_SMD:C_0603_1608Metric_Pad1.08x0.95mm_HandSolder"
 			(at 73.3552 133.35 0)
 			(effects
@@
 			)
 		)
-		(property "Footprint" "Capacitor_SMD:C_0201_0603Metric"
+		(property "Footprint" "Capacitor_SMD:C_0603_1608Metric_Pad1.08x0.95mm_HandSolder"
 			(at 83.5152 133.35 0)
 			(effects

Commit message: BOM Gerbery, schemat w pdfie i zip do oddania na razie bez wszystkich numerów indeksu
Other:
- company: (none) -> Kuba Kulesza, Józef Wiatr, Paweł Laks
- title: (none) -> Złącza
Changed lines of the file:
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@@
 	(generator_version "8.0")
 	(paper "A4")
+	(title_block
+		(title "Złącza")
+		(company "Kuba Kulesza, Józef Wiatr, Paweł Laks")
+	)
 	(junction
 		(at 82.55 124.46)
