File: MCU.kicad_sch (KiCad schematic)
At the start: 22 parts, among them IC1 STM32WBA54KGU6, U1 LTV-817, U2 LTV-817, Y1 TXC 7R-32.000MEEV-T

Commit message: BOM Gerbery, schemat w pdfie i zip do oddania na razie bez wszystkich numerów indeksu
Other:
- company: (none) -> Kuba Kulesza, Józef Wiatr, Paweł Laks
- title: (none) -> Mikrokontroler
Changed lines of the file:
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@@
 	(generator_version "8.0")
 	(paper "A4")
+	(title_block
+		(title "Mikrokontroler")
+		(company "Kuba Kulesza, Józef Wiatr, Paweł Laks")
+	)
 	(junction
 		(at 118.11 147.32)
