File: PSU.kicad_sch (KiCad schematic)
At the start: 1 part, among them U3 IRM-01-3.3

Commit message: BOM Gerbery, schemat w pdfie i zip do oddania na razie bez wszystkich numerów indeksu
Other:
- company: (none) -> Kuba Kulesza, Józef Wiatr, Paweł Laks
- title: (none) -> Zasilanie
Changed lines of the file:
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@@
 	(generator_version "8.0")
 	(paper "A4")
+	(title_block
+		(title "Zasilanie")
+		(company "Kuba Kulesza, Józef Wiatr, Paweł Laks")
+	)
 	(wire
 		(pts
