File: outputs.kicad_sch (KiCad schematic)
At the start: 12 parts, among them Q1 BT136-600, Q2 BT136-600, Q3 MOC3032M, Q4 MOC3032M

Commit message: BOM Gerbery, schemat w pdfie i zip do oddania na razie bez wszystkich numerów indeksu
Other:
- company: (none) -> Kuba Kulesza, Józef Wiatr, Paweł Laks
- title: (none) -> Wyjścia
Changed lines of the file:
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@@
 	(generator_version "8.0")
 	(paper "A4")
+	(title_block
+		(title "Wyjścia")
+		(company "Kuba Kulesza, Józef Wiatr, Paweł Laks")
+	)
 	(junction
 		(at 113.03 62.23)
