File: sterownik_rolety_Zigbee.kicad_sch (KiCad schematic)
At the start: 0 parts

Commit message: BOM Gerbery, schemat w pdfie i zip do oddania na razie bez wszystkich numerów indeksu
Other:
- company: (none) -> Kuba Kulesza, Józef Wiatr, Paweł Laks
- title: (none) -> sterownik rolety z komunikacją zigbee
Changed lines of the file:
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@@
 	(generator_version "8.0")
 	(paper "A4")
+	(title_block
+		(title "sterownik rolety z komunikacją zigbee")
+		(date "2025-01-04")
+		(company "Kuba Kulesza, Józef Wiatr, Paweł Laks")
+	)
 	(sheet
 		(at 124.46 93.98)
